File: eagle/nRF_badge/Badge_03_v4/badge_03v4.brd (EAGLE design)
At the start: 30 x 70 mm, 45 parts, among them J1 PROG_CONN_6, U1 AT25M02, U2 LP2985LV, U3 MCP6231, U4 PCF85263, Y1 32768Hz, Y2 32768Hz

Commit message: Added ULPs to generate BOM and centroid data; post-processed BOM with Digikey part #'s
Parts:
- J1: value PROG_CONN_6 -> (none)
- MIC_F, M_RAW, M_VCC: value TESTPOINT -> (none)
- MK1: value SPU0414(AMP) -> SPU0414
- S1: value JS202011SCQN -> DPDT
- S2: value TACT6MM4 -> TACT6mm
- renumbered MIC to M_RAW, MICVCC to M_VCC
Changed lines of the file:
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@@
 <attribute name="VALUE" x="24.125" y="53.125" size="0.8128" layer="51" font="vector" ratio="16"/>
 </element>
-<element name="MK1" library="Badge" package="MIC_SPU041X" value="SPU0414(AMP)" x="15" y="60.5" smashed="yes" rot="R180">
+<element name="MK1" library="Badge" package="MIC_SPU041X" value="SPU0414" x="15" y="60.5" smashed="yes" rot="R180">
 <attribute name="NAME" x="17.375" y="59.125" size="0.8128" layer="25" font="vector" ratio="16" rot="R180" align="top-right"/>
 </element>
@@
 </element>
 <element name="BAT2" library="Badge" package="BATTCON_20MM_4LEGS_ISO_NOCREAM" value="CR2032" x="15" y="12.25" rot="MR0"/>
-<element name="J1" library="Badge" package="TH_CONN_6" value="PROG_CONN_6" x="3.75" y="55"/>
-<element name="S2" library="Badge" package="TACT1" value="TACT6MM4" x="24.5" y="25.75" smashed="yes">
+<element name="J1" library="Badge" package="TH_CONN_6" value="" x="3.75" y="55"/>
+<element name="S2" library="Badge" package="TACT1" value="TACT6mm" x="24.5" y="25.75" smashed="yes">
 <attribute name="NAME" x="27.5" y="21.5" size="0.8128" layer="25" font="vector" ratio="16" align="bottom-right"/>
 </element>
@@
 <attribute name="VALUE" x="4.375" y="46" size="0.8128" layer="27" font="vector" ratio="16"/>
 </element>
-<element name="S1" library="Badge" package="JS202011SCQN" value="JS202011SCQN" x="15" y="53" smashed="yes">
+<element name="S1" library="Badge" package="JS202011SCQN" value="DPDT" x="15" y="53" smashed="yes">
 <attribute name="NAME" x="13.125" y="57.625" size="0.8128" layer="25" font="vector" ratio="16"/>
 </element>
 <element name="BAT3" library="Badge" package="BU2032SM" value="CR2032" x="15" y="12.25" smashed="yes" rot="MR217"/>
-<element name="MIC" library="Badge" package="TESTPOINT" value="TESTPOINT" x="20" y="62"/>
+<element name="M_RAW" library="Badge" package="TESTPOINT" value="" x="20" y="62"/>
 <element name="C2" library="rcl" package="C0603" value="0u1" x="22.25" y="43.5" smashed="yes">
 <attribute name="NAME" x="19.24" y="43.135" size="0.8128" layer="25" font="vector" ratio="16"/>
@@
 </element>
 <element name="BAT4" library="Badge" package="BU2032SM" value="CR2032" x="15" y="12.25" rot="R323"/>
-<element name="MIC_F" library="Badge" package="TESTPOINT" value="TESTPOINT" x="23.375" y="59"/>
-<element name="MICVCC" library="Badge" package="TESTPOINT" value="TESTPOINT" x="26.125" y="44.625"/>
+<element name="MIC_F" library="Badge" package="TESTPOINT" value="" x="23.375" y="59"/>
+<element name="M_VCC" library="Badge" package="TESTPOINT" value="" x="26.125" y="44.625"/>
 <element name="Y2" library="Badge" package="CRYSTAL_2SMD" value="32768Hz" x="15" y="28.75" smashed="yes" rot="MR0">
 <attribute name="NAME" x="18.25" y="29" size="0.8128" layer="22" font="vector" ratio="16" rot="MR0"/>
@@
 <wire x1="21" y1="61" x2="21.25" y2="61.25" width="0.4064" layer="1"/>
 <wire x1="21.25" y1="61.25" x2="21.9" y2="61" width="0.4064" layer="1"/>
-<contactref element="MIC" pad="P$1"/>
+<contactref element="M_RAW" pad="P$1"/>
 <wire x1="20" y1="62" x2="20" y2="61" width="0.4064" layer="1"/>
 </signal>
@@
 <wire x1="25.5" y1="55" x2="25.55" y2="54.8" width="0.508" layer="1"/>
 <wire x1="25.5" y1="54.25" x2="25.55" y2="54.8" width="0.508" layer="1"/>
-<contactref element="MICVCC" pad="P$1"/>
+<contactref element="M_VCC" pad="P$1"/>
 <wire x1="26.125" y1="44.625" x2="27" y2="45.5" width="0.508" layer="1"/>
 </signal>
