File: eagle/nRF_badge/Badge_03_v4/badge_03v4.brd (EAGLE design)
At the start: 30 x 70 mm, 45 parts, among them U1 AT25M02, U2 LP2985LV, U3 MCP6231, U4 PCF85263, Y1 32768Hz, Y2 32768Hz

Commit message: Fixed Eagle files and re-exported gerbers.
Parts:
- C12: value 0u1 -> 4n7
Changed lines of the file:
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@@
 <attribute name="VALUE" x="16.595" y="40.99" size="0.8128" layer="28" font="vector" ratio="16" rot="MR90"/>
 </element>
-<element name="C12" library="rcl" package="C0603" value="0u1" x="7.5" y="48.375" smashed="yes" rot="R270">
+<element name="C12" library="rcl" package="C0603" value="4n7" x="7.5" y="48.375" smashed="yes" rot="R270">
 <attribute name="NAME" x="6.5" y="50" size="0.8128" layer="25" font="vector" ratio="16"/>
-<attribute name="VALUE" x="6.125" y="46" size="0.8128" layer="27" font="vector" ratio="16"/>
+<attribute name="VALUE" x="6" y="46" size="0.8128" layer="27" font="vector" ratio="16"/>
 </element>
 <element name="C14" library="rcl" package="C0603" value="0u1" x="20.75" y="32.5" smashed="yes" rot="R90">
