File: eagle/nRF_badge/Badge_03_v4/badge_03v4.sch (EAGLE design)
At the start: 45 parts, among them J1 PROG_CONN_6, U1 AT25M02, U2 LP2985LV, U3 MCP6231, U4 PCF85263, Y1 32768Hz, Y2 32768Hz

Commit message: Fixed Eagle files and re-exported gerbers.
Parts:
- C12: value 0u1 -> 4n7
Changed lines of the file:
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@@
 <part name="SUPPLY5" library="Badge" deviceset="VCC" device=""/>
 <part name="SUPPLY6" library="Badge" deviceset="VCC" device=""/>
-<part name="C12" library="rcl" deviceset="C-EU" device="C0603" value="0u1"/>
+<part name="C12" library="rcl" deviceset="C-EU" device="C0603" value="4n7"/>
 <part name="C14" library="rcl" deviceset="C-EU" device="C0603" value="0u1"/>
 <part name="R1" library="rcl" deviceset="R-US_" device="R0603" value="6k8"/>
